File: doc/esp-wroom-32/esp-wroom-32.sch (KiCad schematic (older format))
At the start: 68 parts, among them Q1 MMFT960, Q2 NDT2955, SW1 Power switch, SW2 Jack plugged, U1 4066, U1 ESP32-WROOM, U2 MCP23017_SP, U3 MCP1826 5V, U4 TLP290 / TLP620

Commit message: Further implementation.
Parts:
- added U?: MCP23017_SP, Package_DIP:DIP-28_W7.62mm, symbol Interface_Expansion:MCP23017_SP
Connections:
- wire segments 224 -> 242
