File: doc/esp-wroom-32/esp-wroom-32.sch (KiCad schematic (older format))
At the start: 69 parts, among them Q1 MMFT960, Q2 NDT2955, SW1 Power switch, SW2 Jack plugged, U1 4066, U1 ESP32-WROOM, U2 MCP23017_SP, U3 MCP1826 5V, U3 MCP23017_SP, U4 TLP290 / TLP620

Commit message: Rotary encoder driver fixed.
Parts:
- removed R8: 500, symbol esp-wroom-32-rescue:R-Device
- removed U4: TLP290 / TLP620, ., symbol esp-wroom-32-rescue:TLP290-MEGA2560
- removed U?: VCC, symbol esp-wroom-32-rescue:VCC-power
- removed U?: +BATT, symbol esp-wroom-32-rescue:+BATT-power
- added 100n1: C?, symbol Device:C
- added C2: 100n, symbol Device:C
- added C?: C, symbol Device:C
- added C?: CP, symbol Device:CP
- added U?: AZ1117-3.3, symbol Regulator_Linear:AZ1117-3.3
- gave numbers to parts that had none: 3
- renumbered + to +1, - to -1, . to .1, . to .2, . to .3, . to .4, . to .5, . to .6, 1 to 101, 1 to 102, 1 to 103, 1 to 104, 1 to 105, 3.3V to 3.3V01, Pxx to Pxx1, RF_Module to RF_Module1, ROT_ENC_x to ROT_ENC_x1, SW_xx to SW_xx1
Connections:
- net labels added: GND-power, MCP23017_Input, VCC-power, Vref
- net labels removed: M2560_Input, TX module
Other:
- note added: "Stick Vref"
- note removed: "Flash insulation"
- moved on the sheet: C1, Pxx1

Commit message: Documentation update.
Parts:
- added C?: 100n, symbol Device:C
- added R?: 2k2, symbol Device:R
- added R?: 1K, symbol Device:R
- C?: value C -> 100n
- C?: value CP -> 1u
Connections:
- net labels added: AUDIO, AU_AMPL
- net labels removed: BUZZER
- wire segments 245 -> 250
Other:
- note added: "Audio filter"
Changed lines of the file:
@@
 Rot_2_A
 Text Label 700  4900 0    42   ~ 0
-BUZZER
+AUDIO
 Text Label 4150 7650 1    42   ~ 0
 Rot_2_Push
@@
 U 1 1 5CBFFF64
 P 4800 1400
-F 0 "C?" H 4915 1446 50  0000 L CNN
-F 1 "C" H 4915 1355 50  0000 L CNN
+F 0 "C?" H 4650 1500 50  0000 L CNN
+F 1 "100n" H 4500 1350 50  0000 L CNN
 F 2 "" H 4838 1250 50  0001 C CNN
 F 3 "~" H 4800 1400 50  0001 C CNN
@@
 P 5100 1400
 F 0 "C?" H 5218 1446 50  0000 L CNN
-F 1 "CP" H 5218 1355 50  0000 L CNN
+F 1 "1u" H 5218 1355 50  0000 L CNN
 F 2 "" H 5138 1250 50  0001 C CNN
 F 3 "~" H 5100 1400 50  0001 C CNN
@@
 Text Notes 4200 700  0    60   ~ 0
 Stick Vref
+$Comp
+L Device:R R?
+U 1 1 5CD04313
+P 6050 7300
+F 0 "R?" H 6120 7346 50  0000 L CNN
+F 1 "2k2" H 6120 7255 50  0000 L CNN
+F 2 "" V 5980 7300 50  0001 C CNN
+F 3 "~" H 6050 7300 50  0001 C CNN
+	1    6050 7300
+	1    0    0    -1
+$EndComp
+$Comp
+L Device:R R?
+U 1 1 5CD0446A
+P 6050 6900
+F 0 "R?" H 6120 6946 50  0000 L CNN
+F 1 "1K" H 6120 6855 50  0000 L CNN
+F 2 "" V 5980 6900 50  0001 C CNN
+F 3 "~" H 6050 6900 50  0001 C CNN
+	1    6050 6900
+	1    0    0    -1
+$EndComp
+$Comp
+L power:GND #PWR?
+U 1 1 5CD045A9
+P 6050 7450
+F 0 "#PWR?" H 6050 7200 50  0001 C CNN
+F 1 "GND" H 6055 7277 50  0000 C CNN
+F 2 "" H 6050 7450 50  0001 C CNN
+F 3 "" H 6050 7450 50  0001 C CNN
+	1    6050 7450
+	1    0    0    -1
+$EndComp
+Wire Wire Line
+	6050 7150 6050 7050
+Wire Wire Line
+	5650 6750 6050 6750
+Text Label 5650 6750 0    50   ~ 0
+AUDIO
+$Comp
+L Device:C C?
+U 1 1 5CD6D080
+P 6400 7300
+F 0 "C?" H 6515 7346 50  0000 L CNN
+F 1 "100n" H 6515 7255 50  0000 L CNN
+F 2 "" H 6438 7150 50  0001 C CNN
+F 3 "~" H 6400 7300 50  0001 C CNN
+	1    6400 7300
+	1    0    0    -1
+$EndComp
+Wire Wire Line
+	6400 7150 6050 7150
+Connection ~ 6050 7150
+Wire Wire Line
+	6400 7450 6050 7450
+Connection ~ 6050 7450
+Wire Wire Line
+	6400 7150 6800 7150
+Connection ~ 6400 7150
+Text Label 6500 7150 0    50   ~ 0
+AU_AMPL
+Text Notes 5950 6650 0    60   ~ 0
+Audio filter
 $EndSCHEMATC

Commit message: Some cleanup
Other:
- note added: "Power and PPM managment has not been \nimplemented in firmware.\nSD card SPI needs external pull ups (not drawn)."
Changed lines of the file:
@@
 Text Notes 5950 6650 0    60   ~ 0
 Audio filter
+Text Notes 5300 5950 0    50   ~ 0
+Power and PPM managment has not been \nimplemented in firmware.\nSD card SPI needs external pull ups (not drawn).
 $EndSCHEMATC

Commit message: ESP32 tip set to esp32-2.3-companion
Connections:
- net labels removed: Rot_2_A, Rot_2_B, Rot_2_Push
- wire segments 250 -> 247
Changed lines of the file:
@@
 Text Label 700  4500 0    42   ~ 0
 Stick_LH
-Text Label 3950 7600 1    42   ~ 0
-Rot_2_B
-Text Label 4050 7600 1    42   ~ 0
-Rot_2_A
 Text Label 700  4900 0    42   ~ 0
 AUDIO
-Text Label 4150 7650 1    42   ~ 0
-Rot_2_Push
 Text Label 4450 7650 1    42   ~ 0
 Rot_1_Push
@@
 	4350 7250 4350 7600
 Wire Wire Line
-	3950 7250 3950 7600
-Wire Wire Line
-	4050 7250 4050 7600
-Wire Wire Line
 	3450 7250 3450 7600
 Wire Wire Line
@@
 	4450 7250 4450 7650
 Wire Wire Line
-	4150 7250 4150 7650
-Wire Wire Line
 	5450 3650 5850 3650

Commit message: RF module power control.
Parts:
- removed .4: BUZZER or SPEAKER, symbol esp-wroom-32-rescue:SPEAKER-MEGA2560
- added Q?: NDT2955, symbol esp-wroom-32-rescue:MOSFET_P-MEGA2560
- added Q?: MMFT960, ~, symbol esp-wroom-32-rescue:MOSFET_N-MEGA2560
- added R? (x2): 100K, symbol esp-wroom-32-rescue:R-Device
- added R? (x2): 5.1K, symbol esp-wroom-32-rescue:R-Device
Connections:
- net labels added: RF_POWER, RF_Power, RF_¸VCC
- net labels removed: Buzzer
- wire segments 247 -> 261
Other:
- moved on the sheet: +1, -1, C1, D1, Q1, Q2, R4, R5, R7, SW1, SW2
