File: doc/esp-wroom-32/esp32-WiFi-kit-32.sch (KiCad schematic (older format))
At the start: 32 parts, among them Q1 MMFT960, Q2 NDT2955, SW1 Power switch, U04 +BATT, U05 +BATT, U1 WiFi-kit-32, U2 AZ1117-3.3, U3 MCP23017_SP

Commit message: Updated schematics & cleanup.
Parts:
- added R12: 1K, symbol Device:R_US
- R10: value 5.1K -> 10K
Connections:
- wire segments 118 -> 120
Other:
- note added: "On-module LED \npuls dow with 10K."
- moved on the sheet: 100n1, U1, U3
